File: hardware/pcb/transmitter_sensor_node/Beevil_Node_nRF52840_SX1262.kicad_sch (KiCad schematic)
At the start: 4 parts, among them U1 nRF52840-QIAA, U2 SX1262IMLTRT, U3 TI TMP117 (NIST +-0.08C), U4 TDK ICS-43434 I2S Mic

Commit message: Add Antmicro open-source nRF52840 + Google Coral Edge TPU M.2 hardware KiCad reference designs
Parts:
- U1: footprint (none) -> Package_DFN_QFN:QFN-73-1EP_7x7mm_P0.35mm_EP5.15x5.15mm
- U2: footprint (none) -> Package_DFN_QFN:QFN-24-1EP_4x4mm_P0.5mm_EP2.6x2.6mm
- U3: footprint (none) -> Package_TO_SOT_SMD:SOT-563
- U4: footprint (none) -> Audio:InvenSense_ICS-43434
Changed lines of the file:
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@@
     (property "Reference" "U1" (id 0) (at 100 80 0))
     (property "Value" "nRF52840-QIAA" (id 1) (at 100 85 0))
+    (property "Footprint" "Package_DFN_QFN:QFN-73-1EP_7x7mm_P0.35mm_EP5.15x5.15mm" (id 2) (at 100 90 0))
   )
   (symbol (lib_id "RF_LoRa:SX1262IMLTRT") (at 180 100 0) (unit 1)
@@
     (property "Reference" "U2" (id 0) (at 180 80 0))
     (property "Value" "SX1262IMLTRT" (id 1) (at 180 85 0))
+    (property "Footprint" "Package_DFN_QFN:QFN-24-1EP_4x4mm_P0.5mm_EP2.6x2.6mm" (id 2) (at 180 90 0))
   )
   (symbol (lib_id "Sensor_Temperature:TMP117AIYDCR") (at 100 150 0) (unit 1)
@@
     (property "Reference" "U3" (id 0) (at 100 140 0))
     (property "Value" "TI TMP117 (NIST +-0.08C)" (id 1) (at 100 145 0))
+    (property "Footprint" "Package_TO_SOT_SMD:SOT-563" (id 2) (at 100 148 0))
   )
   (symbol (lib_id "Audio:ICS-43434") (at 180 150 0) (unit 1)
@@
     (property "Reference" "U4" (id 0) (at 180 140 0))
     (property "Value" "TDK ICS-43434 I2S Mic" (id 1) (at 180 145 0))
+    (property "Footprint" "Audio:InvenSense_ICS-43434" (id 2) (at 180 148 0))
   )
 )
